Commit message: Updated confiration for local project

File: lbr_description/urdf/iiwa14_tool/iiwa14_description.xacro (robot description, xacro)
@@ -2,5 +2,5 @@
 <robot xmlns:xacro="http://www.ros.org/wiki/xacro">
     <!-- robot as extracted via https://github.com/syuntoku14/fusion2urdf -->
-    <xacro:macro name="iiwa14"
+    <xacro:macro name="iiwa14_tool"
         params="robot_name:=^|lbr mode:=^|mock system_config_path:=^|'$(find lbr_description)/ros2_control/lbr_system_config.yaml' initial_joint_positions_path:=^|'$(find lbr_description)/ros2_control/initial_joint_positions.yaml'">
         <!-- includes -->
@@ -9,5 +9,5 @@
         <!-- joint limits via yaml -->
         <xacro:property name="joint_limits_path"
-            value="$(find lbr_description)/urdf/iiwa14/joint_limits.yaml" />
+            value="$(find lbr_description)/urdf/iiwa14_tool/joint_limits.yaml" />
         <xacro:property name="joint_limits" value="${xacro.load_yaml(joint_limits_path)}" />
         <!-- constants -->
