Commit message: added urdf for robot with f/t sensor

File: lbr_description/urdf/iiwa_14_FT/iiwa_14_FT.xacro (robot description, xacro)
@@ -4,4 +4,5 @@
     <!-- include the lbr iiwa macro -->
     <xacro:include filename="$(find lbr_description)/urdf/iiwa14/iiwa14_description.xacro" />
+    <xacro:include filename="$(find bota_driver)/urdf/BFT_SENS_ECAT_M8.urdf.xacro" />
     <xacro:arg name="robot_name" default="lbr" />
     <xacro:arg name="mode" default="true" />
@@ -12,4 +13,5 @@
         name="initial_joint_positions_path"
         default="$(find lbr_description)/ros2_control/initial_joint_positions.yaml" />
+    <xacro:arg name="prefix" default="bota_driver_node" />
     <!-- KDL requires a link without inertia / Gazebo requires a connection to world link or robot
     will tipple https://github.com/lbr-stack/lbr_fri_ros2_stack/issues/230 -->
@@ -21,4 +23,9 @@
         <child link="$(arg robot_name)_link_0" />
     </joint>
+    <joint name="bft_sens_ecat_m8_robot_joint" type="fixed">
+        <origin xyz="0 0 0.035" rpy="0 0 3.1415923" />
+        <parent link="$(arg robot_name)_link_7" />
+        <child link="$(arg prefix)_mounting" />
+    </joint>
     <!-- iiwa -->
     <xacro:iiwa14
@@ -27,3 +34,5 @@
         system_config_path="$(arg system_config_path)"
         initial_joint_positions_path="$(arg initial_joint_positions_path)" />
+    <xacro:BFT_SENS_ECAT_M8
+        prefix="$(arg prefix)" />
 </robot>
